File: doc/prototyping-board-schematic/prototyping-board.sch (KiCad schematic (older format))
At the start: 42 parts

Commit message: Prototyping board schematic rev 0.1.1
Parts:
- gave numbers to parts that had none: 42

Commit message: Prototyping board schematic rev 0.1.2
Parts:
- CON1: footprint AVR-ISP-6 -> (none)
- J12: value Pin function select 1A -> Pin function select 1
- J15: value Pin function select 1B -> Pin function select 2
- J24: value Pin function select 2 -> Pin function select 3
Connections:
- net GND: now also R2.1, R3.1, R4.1; no longer R2.2, R3.2, R4.2
- net LED_DRIVE: now also J12.4 (Pin_4), J15.3 (Pin_3); no longer J12.2 (Pin_2), J12.3 (Pin_3)
- net PB0: now also J15.2 (Pin_2); no longer J12.6 (Pin_6)
- net PB2: now also J12.2 (Pin_2); no longer J12.4 (Pin_4)
- net VCC: now also R1.1; no longer J3.1 (Pin_1)
- net at J15.1 (Pin_1): now also R2.2; no longer R2.1
- net at C1.1, J7.2 (Pin_2), SW1.1: now also J3.2 (Pin_2); no longer R1.2
- new net: J12.3 (Pin_3), R3.2
- new net: J12.6 (Pin_6), R4.2
- new net: J3.1 (Pin_1), R1.2
Other:
- moved on the sheet: J12, J15, J3, R1, R2, R3, R4
